Commit message: Separate image processing and driving. Udpate world name. Commit new robot definition.

File: my_robot/urdf/my_robot.xacro (robot description, xacro)
@@ -1,5 +1,12 @@
 <?xml version='1.0'?>
+<!-- Inspired by RX-75-4 Guntank -->
 <robot name="my_robot" xmlns:xacro="http://www.ros.org/wiki/xacro">
   <xacro:include filename="$(find my_robot)/urdf/my_robot.gazebo" />
+   <material name="Guntank Base Blue">
+     <color rgba="0.133 0.2 0.466 1"/>
+   </material>
+   <material name="Guntank Track Grey">
+     <color rgba="0.490 0.509 0.592 1"/>
+   </material>
   <link name="robot_footprint"></link>
   <joint name="robot_footprint_joint" type="fixed">
@@ -9,5 +16,4 @@
   </joint>
   <link name='chassis'>
-    <pose>0 0 0.1 0 0 0</pose>
     <inertial>
       <mass value="15.0"/>
@@ -19,117 +25,275 @@
       />
     </inertial>
-    <collision name='collision'>
-      <origin xyz="0 0 0" rpy=" 0 0 0"/>
-      <geometry>
-        <box size=".4 .2 .1"/>
-      </geometry>
-    </collision>
     <visual name='chassis_visual'>
       <origin xyz="0 0 0" rpy=" 0 0 0"/>
       <geometry>
-        <box size=".4 .2 .1"/>
-      </geometry>
-    </visual>
-    <collision name='back_caster_collision'>
-      <origin xyz="-0.15 0 -0.05" rpy=" 0 0 0"/>
-      <geometry>
-        <sphere radius="0.0499"/>
-      </geometry>
-    </collision>
-    <visual name='back_caster_visual'>
-      <origin xyz="-0.15 0 -0.05" rpy=" 0 0 0"/>
-      <geometry>
-        <sphere radius="0.05"/>
-      </geometry>
-    </visual>
-    <collision name='front_caster_collision'>
-      <origin xyz="0.15 0 -0.05" rpy=" 0 0 0"/>
-      <geometry>
-        <sphere radius="0.0499"/>
-      </geometry>
-    </collision>
-    <visual name='front_caster_visual'>
-      <origin xyz="0.15 0 -0.05" rpy=" 0 0 0"/>
-      <geometry>
-        <sphere radius="0.05"/>
-      </geometry>
-    </visual>
+        <box size="0.5 0.4 0.2"/>
+      </geometry>
+      <material name="Guntank Base Blue"/>
+    </visual>
+    <collision name='collision'>
+      <origin xyz="0 0 0" rpy=" 0 0 0"/>
+      <geometry>
+        <box size="0.5 0.4 0.2"/>
+      </geometry>
+    </collision>
   </link>
   <link name='left_wheel'>
     <inertial>
       <mass value="5.0"/>
-      <origin xyz="0.0 0 0" rpy=" 0 0 0"/>
-      <inertia
-          ixx="0.1" ixy="0" ixz="0"
-          iyy="0.1" iyz="0"
-          izz="0.1"
-      />
-    </inertial>
-    <collision name='collision'>
+      <origin xyz="0 0 0" rpy="0 1.5707 1.5707"/>
+      <inertia
+          ixx="0.1" ixy="0" ixz="0"
+          iyy="0.1" iyz="0"
+          izz="0.1"
+      />
+    </inertial>
+    <visual name='left_wheel_visual'>
+      <origin xyz="0 0 0" rpy="0 1.5707 1.5707"/>
+      <geometry>
+        <cylinder radius="0.05" length="0.075"/>
+      </geometry>
+      <material name="Guntank Track Grey"/>
+    </visual>
+    <collision name='collision'>
+      <origin xyz="0 0 0" rpy="0 1.5707 1.5707"/>
+      <geometry>
+        <cylinder radius="0.05" length="0.075"/>
+      </geometry>
+    </collision>
+  </link>
+  <joint type="continuous" name="left_wheel_hinge">
+    <origin xyz="0 0.2375 -0.128" rpy="0 0 0"/>
+    <child link="left_wheel"/>
+    <parent link="chassis"/>
+    <axis xyz="0 1 0" rpy="0 0 0"/>
+    <limit effort="10000" velocity="1000"/>
+    <dynamics damping="0" friction="0"/>
+  </joint>
+  <link name='left_back_road_wheel'>
+    <inertial>
+      <mass value="5.0"/>
+      <origin xyz="0 0 0" rpy="0 1.5707 1.5707"/>
+      <inertia
+          ixx="0.1" ixy="0" ixz="0"
+          iyy="0.1" iyz="0"
+          izz="0.1"
+      />
+    </inertial>
+    <visual name='left_back_road_wheel_visual'>
+      <origin xyz="0 0 0" rpy="0 1.5707 1.5707"/>
+      <geometry>
+        <cylinder radius="0.05" length="0.075"/>
+      </geometry>
+      <material name="Guntank Track Grey"/>
+    </visual>
+    <collision name='collision'>
+      <origin xyz="0 0 0" rpy="0 1.5707 1.5707"/>
+      <geometry>
+        <cylinder radius="0.05" length="0.075"/>
+      </geometry>
+    </collision>
+  </link>
+  <joint type="continuous" name="left_back_road_wheel_hinge">
+    <origin xyz="-0.2 0.2375 -0.128" rpy="0 0 0"/>
+    <child link="left_back_road_wheel"/>
+    <parent link="chassis"/>
+    <axis xyz="0 1 0" rpy="0 0 0"/>
+    <limit effort="10000" velocity="1000"/>
+    <dynamics damping="0.0" friction="0.0"/>
+  </joint>
+  <link name='left_front_road_wheel'>
+    <inertial>
+      <mass value="5.0"/>
+      <origin xyz="0 0 0" rpy="0 1.5707 1.5707"/>
+      <inertia
+          ixx="0.1" ixy="0" ixz="0"
+          iyy="0.1" iyz="0"
+          izz="0.1"
+      />
+    </inertial>
+    <visual name='left_front_road_wheel_visual'>
+      <origin xyz="0 0 0" rpy="0 1.5707 1.5707"/>
+      <geometry>
+        <cylinder radius="0.05" length="0.075"/>
+      </geometry>
+      <material name="Guntank Track Grey"/>
+    </visual>
+    <collision name='collision'>
+      <origin xyz="0 0 0" rpy="0 1.5707 1.5707"/>
+      <geometry>
+        <cylinder radius="0.05" length="0.075"/>
+      </geometry>
+    </collision>
+  </link>
+  <joint type="continuous" name="left_front_road_wheel_hinge">
+    <origin xyz="0.2 0.2375 -0.128" rpy="0 0 0"/>
+    <child link="left_front_road_wheel"/>
+    <parent link="chassis"/>
+    <axis xyz="0 1 0" rpy="0 0 0"/>
+    <limit effort="10000" velocity="1000"/>
+    <dynamics damping="0.0" friction="0.0"/>
+  </joint>
+  <link name='left_return_roller'>
+    <inertial>
+      <mass value="5.0"/>
+      <origin xyz="0 0 0" rpy="0 1.5707 1.5707"/>
+      <inertia
+          ixx="0.1" ixy="0" ixz="0"
+          iyy="0.1" iyz="0"
+          izz="0.1"
+      />
+    </inertial>
+    <visual name='left_return_roller_visual'>
+      <origin xyz="0 0 0" rpy="0 1.5707 1.5707"/>
+      <geometry>
+        <cylinder radius="0.05" length="0.075"/>
+      </geometry>
+      <material name="Guntank Track Grey"/>
+    </visual>
+    <collision name='collision'>
+      <origin xyz="0 0 0" rpy="0 1.5707 1.5707"/>
+      <geometry>
+        <cylinder radius="0.05" length="0.075"/>
+      </geometry>
+    </collision>
+  </link>
+  <joint type="continuous" name="left_return_roller_hinge">
+    <origin xyz="0.1 0.2375 0.03" rpy="0 0 0"/>
+    <child link="left_return_roller"/>
+    <parent link="chassis"/>
+    <axis xyz="0 1 0" rpy="0 0 0"/>
+    <limit effort="10000" velocity="1000"/>
+    <dynamics damping="0.0" friction="0.0"/>
+  </joint>
+  <link name='right_wheel'>
+    <inertial>
+      <mass value="5.0"/>
+      <origin xyz="0 0 0" rpy="0 1.5707 1.5707"/>
+      <inertia
+          ixx="0.1" ixy="0" ixz="0"
+          iyy="0.1" iyz="0"
+          izz="0.1"
+      />
+    </inertial>
+    <visual name='right_wheel_visual'>
       <origin xyz="0 0 0" rpy=" 0 1.5707 1.5707"/>
       <geometry>
-        <cylinder radius="0.1" length="0.05"/>
-      </geometry>
-    </collision>
-    <visual name='chassis_visual'>
+        <cylinder radius="0.05" length="0.075"/>
+      </geometry>
+      <material name="Guntank Track Grey"/>
+    </visual>
+    <collision name='collision'>
       <origin xyz="0 0 0" rpy=" 0 1.5707 1.5707"/>
       <geometry>
-        <cylinder radius="0.1" length="0.05"/>
-      </geometry>
-    </visual>
-  </link>
-  <joint type="continuous" name="left_wheel_hinge">
-    <origin xyz="0 0.15 0" rpy="0 0 0"/>
-    <child link="left_wheel"/>
-    <parent link="chassis"/>
-    <axis xyz="0 1 0" rpy="0 0 0"/>
-    <limit effort="10000" velocity="1000"/>
-    <dynamics damping="1.0" friction="1.0"/>
-  </joint>
-  <link name='right_wheel'>
-    <inertial>
-      <mass value="5.0"/>
-      <origin xyz="0.0 0 0" rpy=" 0 0 0"/>
-      <inertia
-          ixx="0.1" ixy="0" ixz="0"
-          iyy="0.1" iyz="0"
-          izz="0.1"
-      />
-    </inertial>
-    <collision name='collision'>
-      <origin xyz="0 0 0" rpy=" 0 1.5707 1.5707"/>
-      <geometry>
-        <cylinder radius="0.1" length="0.05"/>
-      </geometry>
-    </collision>
-    <visual name='chassis_visual'>
-      <origin xyz="0 0 0" rpy=" 0 1.5707 1.5707"/>
-      <geometry>
-        <cylinder radius="0.1" length="0.05"/>
-      </geometry>
-    </visual>
+        <cylinder radius="0.05" length="0.075"/>
+      </geometry>
+    </collision>
   </link>
   <joint type="continuous" name="right_wheel_hinge">
-    <origin xyz="0 -0.15 0" rpy="0 0 0"/>
+    <origin xyz="0 -0.2375 -0.128" rpy="0 0 0"/>
     <child link="right_wheel"/>
     <parent link="chassis"/>
     <axis xyz="0 1 0" rpy="0 0 0"/>
     <limit effort="10000" velocity="1000"/>
-    <dynamics damping="1.0" friction="1.0"/>
+    <dynamics damping="0" friction="0"/>
+  </joint>
+  <link name='right_back_road_wheel'>
+    <inertial>
+      <mass value="5.0"/>
+      <origin xyz="0 0 0" rpy="0 1.5707 1.5707"/>
+      <inertia
+          ixx="0.1" ixy="0" ixz="0"
+          iyy="0.1" iyz="0"
+          izz="0.1"
+      />
+    </inertial>
+    <visual name='right_back_road_wheel_visual'>
+      <origin xyz="0 0 0" rpy="0 1.5707 1.5707"/>
+      <geometry>
+        <cylinder radius="0.05" length="0.075"/>
+      </geometry>
+      <material name="Guntank Track Grey"/>
+    </visual>
+    <collision name='collision'>
+      <origin xyz="0 0 0" rpy="0 1.5707 1.5707"/>
+      <geometry>
+        <cylinder radius="0.05" length="0.075"/>
+      </geometry>
+    </collision>
+  </link>
+  <joint type="continuous" name="right_back_road_wheel_hinge">
+    <origin xyz="-0.2 -0.2375 -0.128" rpy="0 0 0"/>
+    <child link="right_back_road_wheel"/>
+    <parent link="chassis"/>
+    <axis xyz="0 1 0" rpy="0 0 0"/>
+    <limit effort="10000" velocity="1000"/>
+    <dynamics damping="0.0" friction="0.0"/>
+  </joint>
+  <link name='right_front_road_wheel'>
+    <inertial>
+      <mass value="5.0"/>
+      <origin xyz="0 0 0" rpy="0 1.5707 1.5707"/>
+      <inertia
+          ixx="0.1" ixy="0" ixz="0"
+          iyy="0.1" iyz="0"
+          izz="0.1"
+      />
+    </inertial>
+    <visual name='right_front_road_wheel_visual'>
+      <origin xyz="0 0 0" rpy="0 1.5707 1.5707"/>
+      <geometry>
+        <cylinder radius="0.05" length="0.075"/>
+      </geometry>
+      <material name="Guntank Track Grey"/>
+    </visual>
+    <collision name='collision'>
+      <origin xyz="0 0 0" rpy="0 1.5707 1.5707"/>
+      <geometry>
+        <cylinder radius="0.05" length="0.075"/>
+      </geometry>
+    </collision>
+  </link>
+  <joint type="continuous" name="right_front_road_wheel_hinge">
+    <origin xyz="0.2 -0.2375 -0.128" rpy="0 0 0"/>
+    <child link="right_front_road_wheel"/>
+    <parent link="chassis"/>
+    <axis xyz="0 1 0" rpy="0 0 0"/>
+    <limit effort="10000" velocity="1000"/>
+    <dynamics damping="0.0" friction="0.0"/>
+  </joint>
+  <link name='right_return_roller'>
+    <inertial>
+      <mass value="5.0"/>
+      <origin xyz="0 0 0" rpy="0 1.5707 1.5707"/>
+      <inertia
+          ixx="0.1" ixy="0" ixz="0"
+          iyy="0.1" iyz="0"
+          izz="0.1"
+      />
+    </inertial>
+    <visual name='right_return_roller_visual'>
+      <origin xyz="0 0 0" rpy="0 1.5707 1.5707"/>
+      <geometry>
+        <cylinder radius="0.05" length="0.075"/>
+      </geometry>
+      <material name="Guntank Track Grey"/>
+    </visual>
+    <collision name='collision'>
+      <origin xyz="0 0 0" rpy="0 1.5707 1.5707"/>
+      <geometry>
+        <cylinder radius="0.05" length="0.075"/>
+      </geometry>
+    </collision>
+  </link>
+  <joint type="continuous" name="right_return_roller_hinge">
+    <origin xyz="0.1 -0.2375 0.03" rpy="0 0 0"/>
+    <child link="right_return_roller"/>
+    <parent link="chassis"/>
+    <axis xyz="0 1 0" rpy="0 0 0"/>
+    <limit effort="10000" velocity="1000"/>
+    <dynamics damping="0.0" friction="0.0"/>
   </joint>
   <link name='camera'>
-    <pose>0 0 0 0 0 0</pose>
-    <visual name='camera_visual'>
-      <origin xyz="0 0 0" rpy=" 0 0 0"/>
-      <geometry>
-        <box size="0.05 0.05 0.05"/>
-      </geometry>
-    </visual>
-    <collision name='camera_collision'>
-      <origin xyz="0 0 0" rpy=" 0 0 0"/>
-      <geometry>
-        <box size="0.05 0.05 0.05"/>
-      </geometry>
-    </collision>
     <inertial>
       <mass value="0.1"/>
@@ -141,7 +305,19 @@
       />
     </inertial>
+    <visual name='camera_visual'>
+      <origin xyz="0 0 0" rpy=" 0 0 0"/>
+      <geometry>
+        <box size="0.05 0.05 0.05"/>
+      </geometry>
+    </visual>
+    <collision name='camera_collision'>
+      <origin xyz="0 0 0" rpy=" 0 0 0"/>
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
Commit message: Update build order. Somehow building from scratch will not build the service first. Update drive controller update rate. Add material to the guntank base. Added variable rotation speed based on distance.

File: my_robot/urdf/my_robot.xacro (robot description, xacro)
@@ -3,10 +3,30 @@
 <robot name="my_robot" xmlns:xacro="http://www.ros.org/wiki/xacro">
   <xacro:include filename="$(find my_robot)/urdf/my_robot.gazebo" />
-   <material name="Guntank Base Blue">
-     <color rgba="0.133 0.2 0.466 1"/>
-   </material>
-   <material name="Guntank Track Grey">
-     <color rgba="0.490 0.509 0.592 1"/>
-   </material>
+  <xacro:macro name="material_GuntankBaseBlue">
+    <visual>
+      <material>
+        <ambient>0.133 0.2 0.466 1</ambient>
+        <diffuse>0.133 0.2 0.466 1</diffuse>
+        <specular>0.1 0.1 0.1 1</specular>
+        <emissive>0 0 0 0</emissive>
+      </material>
+    </visual>
+  </xacro:macro>
+  <material name="Guntank Base Blue">
+    <color rgba="0.133 0.2 0.466 1"/>
+  </material>
+  <xacro:macro name="material_GuntankTrackGrey">
+    <visual>
+      <material>
+        <ambient>0.490 0.509 0.592 1</ambient>
+        <diffuse>0.490 0.509 0.592 1</diffuse>
+        <specular>0.1 0.1 0.1 1</specular>
+        <emissive>0 0 0 0</emissive>
+      </material>
+    </visual>
+  </xacro:macro>
+  <material name="Guntank Track Grey">
+    <color rgba="0.490 0.509 0.592 1"/>
+  </material>
   <link name="robot_footprint"></link>
   <joint name="robot_footprint_joint" type="fixed">
@@ -39,4 +59,7 @@
     </collision>
   </link>
+  <gazebo reference="chassis">
+    <xacro:material_GuntankBaseBlue />
+  </gazebo>
   <link name='left_wheel'>
     <inertial>
@@ -63,4 +86,7 @@
     </collision>
   </link>
+  <gazebo reference="left_wheel">
+    <xacro:material_GuntankTrackGrey />
+  </gazebo>
   <joint type="continuous" name="left_wheel_hinge">
     <origin xyz="0 0.2375 -0.128" rpy="0 0 0"/>
@@ -95,4 +121,7 @@
     </collision>
   </link>
+  <gazebo reference="left_back_road_wheel">
+    <xacro:material_GuntankTrackGrey />
+  </gazebo>
   <joint type="continuous" name="left_back_road_wheel_hinge">
     <origin xyz="-0.2 0.2375 -0.128" rpy="0 0 0"/>
@@ -101,5 +130,5 @@
     <axis xyz="0 1 0" rpy="0 0 0"/>
     <limit effort="10000" velocity="1000"/>
-    <dynamics damping="0.0" friction="0.0"/>
+    <dynamics damping="1.0" friction="1.0"/>
   </joint>
   <link name='left_front_road_wheel'>
@@ -127,4 +156,7 @@
     </collision>
   </link>
+  <gazebo reference="left_front_road_wheel">
+    <xacro:material_GuntankTrackGrey />
+  </gazebo>
   <joint type="continuous" name="left_front_road_wheel_hinge">
     <origin xyz="0.2 0.2375 -0.128" rpy="0 0 0"/>
@@ -133,5 +165,5 @@
     <axis xyz="0 1 0" rpy="0 0 0"/>
     <limit effort="10000" velocity="1000"/>
-    <dynamics damping="0.0" friction="0.0"/>
+    <dynamics damping="1.0" friction="1.0"/>
   </joint>
   <link name='left_return_roller'>
@@ -159,4 +191,7 @@
     </collision>
   </link>
+  <gazebo reference="left_return_roller">
+    <xacro:material_GuntankTrackGrey />
+  </gazebo>
   <joint type="continuous" name="left_return_roller_hinge">
     <origin xyz="0.1 0.2375 0.03" rpy="0 0 0"/>
@@ -191,4 +226,7 @@
     </collision>
   </link>
+  <gazebo reference="right_wheel">
+    <xacro:material_GuntankTrackGrey />
+  </gazebo>
   <joint type="continuous" name="right_wheel_hinge">
     <origin xyz="0 -0.2375 -0.128" rpy="0 0 0"/>
@@ -223,4 +261,7 @@
     </collision>
   </link>
+  <gazebo reference="right_back_road_wheel">
+    <xacro:material_GuntankTrackGrey />
+  </gazebo>
   <joint type="continuous" name="right_back_road_wheel_hinge">
     <origin xyz="-0.2 -0.2375 -0.128" rpy="0 0 0"/>
@@ -229,5 +270,5 @@
     <axis xyz="0 1 0" rpy="0 0 0"/>
     <limit effort="10000" velocity="1000"/>
-    <dynamics damping="0.0" friction="0.0"/>
+    <dynamics damping="1.0" friction="1.0"/>
   </joint>
   <link name='right_front_road_wheel'>
@@ -255,4 +296,7 @@
     </collision>
   </link>
+  <gazebo reference="right_front_road_wheel">
+    <xacro:material_GuntankTrackGrey />
+  </gazebo>
   <joint type="continuous" name="right_front_road_wheel_hinge">
     <origin xyz="0.2 -0.2375 -0.128" rpy="0 0 0"/>
@@ -261,5 +305,5 @@
     <axis xyz="0 1 0" rpy="0 0 0"/>
     <limit effort="10000" velocity="1000"/>
-    <dynamics damping="0.0" friction="0.0"/>
+    <dynamics damping="1.0" friction="1.0"/>
   </joint>
   <link name='right_return_roller'>
@@ -287,4 +331,7 @@
     </collision>
   </link>
+  <gazebo reference="right_return_roller">
+    <xacro:material_GuntankTrackGrey />
+  </gazebo>
   <joint type="continuous" name="right_return_roller_hinge">
     <origin xyz="0.1 -0.2375 0.03" rpy="0 0 0"/>

Commit message: Try to implement a dynamic solid colored ball finder.

File: my_robot/urdf/my_robot.xacro (robot description, xacro)
@@ -366,5 +366,5 @@
   </link>
   <joint type="fixed" name="camera_joint">
-    <origin xyz="0.275 0 0" rpy="0 0 0"/>
+    <origin xyz="0.275 0 -0.075" rpy="0 0 0"/>
     <child link="camera"/>
     <parent link="chassis"/>

Commit message: my_robot/config/* my_robot/launch/* my_robot/maps/* 1. Implement localization using AMCL.
my_robot.xacro
1. Moved the middle road wheel up to try to avoid any unusual behavior.

japariparkv2.world
1. Moved the world to make sure the origin point is empty

File: my_robot/urdf/my_robot.xacro (robot description, xacro)
@@ -90,5 +90,5 @@
   </gazebo>
   <joint type="continuous" name="left_wheel_hinge">
-    <origin xyz="0 0.2375 -0.128" rpy="0 0 0"/>
+    <origin xyz="0 0.2375 -0.1" rpy="0 0 0"/>
     <child link="left_wheel"/>
     <parent link="chassis"/>
@@ -230,5 +230,5 @@
   </gazebo>
   <joint type="continuous" name="right_wheel_hinge">
-    <origin xyz="0 -0.2375 -0.128" rpy="0 0 0"/>
+    <origin xyz="0 -0.2375 -0.1" rpy="0 0 0"/>
     <child link="right_wheel"/>
     <parent link="chassis"/>

Commit message: config/* 1. Adjust to try and make the nav a bit smoother.
amcl.launch
1. Update values.

japaraiparkv2.pgm
1. Adjusted some more positions.

my_robot.xacro
1. Moved the hakuyo sensor a bit to the front.

File: my_robot/urdf/my_robot.xacro (robot description, xacro)
@@ -395,5 +395,5 @@
   </link>
   <joint type="fixed" name="hokuyo_joint">
-    <origin xyz="0.2 0 0.125" rpy="0 0 0"/>
+    <origin xyz="0.21 0 0.125" rpy="0 0 0"/>
     <child link="hokuyo"/>
     <parent link="chassis"/>

Commit message: Added launch files for mapping and teleop. Added body part of the guntank. Added the RGB-D camera for mapping. Modified the camera plugin to use the Kinect obj file and the necessary params. Added the generated DB of japariparkv2.

File: my_robot/urdf/my_robot.xacro (robot description, xacro)
@@ -62,4 +62,37 @@
     <xacro:material_GuntankBaseBlue />
   </gazebo>
+  <link name='body'>
+    <inertial>
+      <mass value="5.0"/>
+      <origin xyz="0.0 0 0" rpy=" 0 0 0"/>
+      <inertia
+          ixx="0.1" ixy="0" ixz="0"
+          iyy="0.1" iyz="0"
+          izz="0.1"
+      />
+    </inertial>
+    <visual name='body_visual'>
+      <origin xyz="0 0 0" rpy=" 0 0 0"/>
+      <geometry>
+        <box size="0.15 0.25 0.25"/>
+      </geometry>
+      <material name="Guntank Base Blue"/>
+    </visual>
+    <collision name='collision'>
+      <origin xyz="0 0 0" rpy=" 0 0 0"/>
+      <geometry>
+        <box size="0.15 0.25 0.25"/>
+      </geometry>
+    </collision>
+  </link>
+  <gazebo reference="body">
+    <xacro:material_GuntankBaseBlue />
+  </gazebo>
+  <!-- Fixed joint for now -->
+  <joint type="fixed" name="body_hinge">
+    <origin xyz="0 0 0.225" rpy="0 0 0"/>
+    <child link="body"/>
+    <parent link="chassis"/>
+  </joint>
   <link name='left_wheel'>
     <inertial>
@@ -400,3 +433,17 @@
     <axis xyz="0 1 0" rpy="0 0 0"/>
   </joint>
+  <link name="camera_link_optical">
+    <!--<visual name='camera_visual'>
+      <origin xyz="0 0 0" rpy=" 0 0 0"/>
+      <geometry>
+        <box size="0.05 0.05 0.05"/>
+      </geometry>
+    </visual>-->
+  </link>
+  <joint name="camera_optical_joint" type="fixed">
+    <origin xyz="0.075 0 0.125" rpy="0 0 0"/>
+    <parent link="body"/>
+    <child link="camera_link_optical"/>
+    <axis xyz="0 1 0" rpy="0 0 0"/>
+  </joint>
 </robot>
